File: ControlBoard.sch (EAGLE design)
At the start: 2 parts, among them J1 47053-1000, U1 ARDUINO_PRO_MINI

Commit message: Made the first version of the pcb
Parts:
- removed U1: ARDUINO_PRO_MINI, ARDUINO_PRO_MINI:ARDUINO_PRO_MINI
- added 12VBATTERY, PELTIER: B2B-XH-A(LF)(SN), B2B-XH-A_LF__SN_:B2B-XH-A(LF)(SN)
- added ARDUINO-NANO: ABX00028, ABX00028:ABX00028
- added ICMOSFET: RFP30N06LE, RFP30N06LE:RFP30N06LE
- added ICOPAMP: LM358, LM358:LM358
- added R1: 1Ω, adafruit:FLIPFLOP-RES
- renumbered J1 to FAN
Connections:
- new net IREGULATOR: ICMOSFET.D, PELTIER.2
- new net N$1: ICMOSFET.S, ICOPAMPG1.-IN, R1.1
- new net N$5: ICMOSFET.G, ICOPAMPG1.OUT
- new net PELTIERCONTROL: ARDUINO-NANO.A1, ICOPAMPG1.+IN
- net 12V: now also 12VBATTERY.1, ARDUINO-NANO.VIN, PELTIER.1
- net GND: now also 12VBATTERY.2, ARDUINO-NANO.GND, R1.2
- net PWM: now also ARDUINO-NANO.D3/PWM; no longer U1.D3

Commit message: Cleaned a bit of the pcb and addded the tmp36 thermocouple
Parts:
- added TMP36: B3B-XH-A(LF)(SN), B3B-XH-A_LF__SN_:B3B-XH-A(LF)(SN)
Connections:
- new net 5V: ARDUINO-NANO.+5V, TMP36.1
- new net THERMOCOUPLE: ARDUINO-NANO.A3, TMP36.2
- net GND: now also TMP36.3
Changed lines of the file:
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@@
 <part name="12VBATTERY" library="B2B-XH-A_LF__SN_" deviceset="B2B-XH-A(LF)(SN)" device=""/>
 <part name="PELTIER" library="B2B-XH-A_LF__SN_" deviceset="B2B-XH-A(LF)(SN)" device=""/>
+<part name="TMP36" library="B3B-XH-A_LF__SN_" deviceset="B3B-XH-A(LF)(SN)" device=""/>
 </parts>
 <sheets>
@@
 <attribute name="VALUE" x="60.96" y="58.42" size="1.778" layer="96"/>
 </instance>
+<instance part="TMP36" gate="G$1" x="124.46" y="33.02" smashed="yes">
+<attribute name="NAME" x="119.38" y="38.862" size="1.778" layer="95"/>
+<attribute name="VALUE" x="119.38" y="25.4" size="1.778" layer="96"/>
+</instance>
 </instances>
 <busses>
@@
 <wire x1="48.26" y1="33.02" x2="48.26" y2="27.94" width="0.1524" layer="91"/>
 <label x="48.26" y="25.4" size="1.778" layer="95"/>
+</segment>
+<segment>
+<pinref part="TMP36" gate="G$1" pin="3"/>
+<wire x1="114.3" y1="30.48" x2="109.22" y2="30.48" width="0.1524" layer="91"/>
+<wire x1="109.22" y1="30.48" x2="109.22" y2="25.4" width="0.1524" layer="91"/>
+<label x="109.22" y="22.86" size="1.778" layer="95"/>
 </segment>
 </net>
@@
 </segment>
 </net>
+<net name="5V" class="0">
+<segment>
+<pinref part="TMP36" gate="G$1" pin="1"/>
+<wire x1="114.3" y1="35.56" x2="104.14" y2="35.56" width="0.1524" layer="91"/>
+<label x="104.14" y="38.1" size="1.778" layer="95"/>
+</segment>
+<segment>
+<pinref part="ARDUINO-NANO" gate="G$1" pin="+5V"/>
+<wire x1="10.16" y1="58.42" x2="27.94" y2="58.42" width="0.1524" layer="91"/>
+<label x="27.94" y="60.96" size="1.778" layer="95"/>
+</segment>
+</net>
+<net name="THERMOCOUPLE" class="0">
+<segment>
+<pinref part="ARDUINO-NANO" gate="G$1" pin="A3"/>
+<wire x1="-30.48" y1="35.56" x2="-45.72" y2="35.56" width="0.1524" layer="91"/>
+<wire x1="-45.72" y1="35.56" x2="-45.72" y2="33.02" width="0.1524" layer="91"/>
+<label x="-53.34" y="30.48" size="1.778" layer="95"/>
+</segment>
+<segment>
+<pinref part="TMP36" gate="G$1" pin="2"/>
+<wire x1="114.3" y1="33.02" x2="96.52" y2="33.02" width="0.1524" layer="91"/>
+<label x="88.9" y="33.02" size="1.778" layer="95"/>
+</segment>
+</net>
